File: SFP.kicad_sch (KiCad schematic)
At the start: 1 part, among them J2 SFPK-SL

Commit message: update capacitor part numbers
Parts:
- J2: MPN SFPK-SL -> SFPK-SL
Changed lines of the file:
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@@
 			)
 		)
-		(property "MPN" "  SFPK-SL"
+		(property "MPN" "SFPK-SL"
 			(at 132.08 64.77 0)
 			(effects

Commit message: Change part numbers for nextpcb
Parts:
- J2: Comment (none) -> Cage shell is Mfr Part#: HC-SFP-01L; MANUFACTURER Samtec -> HCTL; MPN SFPK-SL -> HC-SFP-20P
Changed lines of the file:
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@@
 			)
 		)
-		(property "MANUFACTURER" "Samtec"
+		(property "MANUFACTURER" "HCTL"
 			(at 132.08 64.77 0)
 			(effects
@@
 			)
 		)
-		(property "MPN" "SFPK-SL"
+		(property "MPN" "HC-SFP-20P"
 			(at 132.08 64.77 0)
 			(effects
+				(font
+					(size 1.27 1.27)
+				)
+				(hide yes)
+			)
+		)
+		(property "Comment" "Cage shell is Mfr Part#: HC-SFP-01L"
+			(at 132.08 64.77 0)
+			(effects

Commit message: modify title block
Other:
- company: (none) -> MicroRidge Technology LTD
- title: (none) -> FMC-SFP
Changed lines of the file:
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@@
 	(generator_version "8.0")
 	(paper "A4")
+	(title_block
+		(title "FMC-SFP")
+		(date "2024-05-08")
+		(rev "Rev0")
+		(company "MicroRidge Technology LTD")
+	)
 	(junction
 		(at 148.59 82.55)
