File: SFP.kicad_sch (KiCad schematic)
At the start: 1 part, among them J2 SFPK-SL

Commit message: modify title block
Other:
- company: (none) -> MicroRidge Technology LTD
- title: (none) -> FMC-SFP
Changed lines of the file:
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@@
 	(generator_version "8.0")
 	(paper "A4")
+	(title_block
+		(title "FMC-SFP")
+		(date "2024-05-08")
+		(rev "Rev0")
+		(company "MicroRidge Technology LTD")
+	)
 	(junction
 		(at 148.59 82.55)
