File: SFP.kicad_sch (KiCad schematic)
At the start: 22 parts, among them J2 SFP+, J3 132134, J4 132134, U1 MAX9113EKA_TT, U4 TXS0108EPW

Commit message: Update layout with i2c
Parts:
- C6, C8: footprint (none) -> Capacitor_SMD:C_0603_1608Metric; MANUFACTURER (none) -> KEMET; MPN (none) -> C0603C104M5RAC7867
- R14, R16, R27, R28: MANUFACTURER (none) -> UNI-ROYAL(Uniroyal Elec); MPN (none) -> 0805W8F1001T5E
Changed lines of the file:
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@@
 			)
 		)
-		(property "Footprint" ""
+		(property "Footprint" "Capacitor_SMD:C_0603_1608Metric"
 			(at 171.7548 104.14 0)
 			(effects
@@
 		)
 		(property "Description" "Unpolarized capacitor"
+			(at 172.72 100.33 0)
+			(effects
+				(font
+					(size 1.27 1.27)
+				)
+				(hide yes)
+			)
+		)
+		(property "MANUFACTURER" "KEMET"
+			(at 172.72 100.33 0)
+			(effects
+				(font
+					(size 1.27 1.27)
+				)
+				(hide yes)
+			)
+		)
+		(property "MPN" "C0603C104M5RAC7867"
 			(at 172.72 100.33 0)
 			(effects
@@
 			)
 		)
-		(property "MANUFACTURER" ""
+		(property "MANUFACTURER" "UNI-ROYAL(Uniroyal Elec) "
 			(at 222.25 110.49 0)
 			(effects
@@
 			)
 		)
-		(property "MPN" ""
+		(property "MPN" "0805W8F1001T5E"
 			(at 222.25 110.49 0)
 			(effects
@@
 			)
 		)
-		(property "Footprint" ""
+		(property "Footprint" "Capacitor_SMD:C_0603_1608Metric"
 			(at 204.7748 104.14 0)
 			(effects
@@
 		)
 		(property "Description" "Unpolarized capacitor"
+			(at 205.74 100.33 0)
+			(effects
+				(font
+					(size 1.27 1.27)
+				)
+				(hide yes)
+			)
+		)
+		(property "MANUFACTURER" "KEMET"
+			(at 205.74 100.33 0)
+			(effects
+				(font
+					(size 1.27 1.27)
+				)
+				(hide yes)
+			)
+		)
+		(property "MPN" "C0603C104M5RAC7867"
 			(at 205.74 100.33 0)
 			(effects
@@
 			)
 		)
-		(property "MANUFACTURER" ""
+		(property "MANUFACTURER" "UNI-ROYAL(Uniroyal Elec) "
 			(at 153.67 109.22 0)
 			(effects
@@
 			)
 		)
-		(property "MPN" ""
+		(property "MPN" "0805W8F1001T5E"
 			(at 153.67 109.22 0)
 			(effects
@@
 			)
 		)
-		(property "MANUFACTURER" ""
+		(property "MANUFACTURER" "UNI-ROYAL(Uniroyal Elec) "
 			(at 161.29 109.22 0)
 			(effects
@@
 			)
 		)
-		(property "MPN" ""
+		(property "MPN" "0805W8F1001T5E"
 			(at 161.29 109.22 0)
 			(effects
@@
 			)
 		)
-		(property "MANUFACTURER" ""
+		(property "MANUFACTURER" "UNI-ROYAL(Uniroyal Elec) "
 			(at 214.63 110.49 0)
 			(effects
@@
 			)
 		)
-		(property "MPN" ""
+		(property "MPN" "0805W8F1001T5E"
 			(at 214.63 110.49 0)
 			(effects

Commit message: add level shifter Part Number
Parts:
- U4: MANUFACTURER (none) -> Texas Instruments; MPN (none) -> TXS0108EPW
Changed lines of the file:
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@@
+			)
+		)
+		(property "MANUFACTURER" "Texas Instruments"
+			(at 185.42 124.46 0)
+			(effects
+				(font
+					(size 1.27 1.27)
+				)
+				(hide yes)
+			)
+		)
+		(property "MPN" "TXS0108EPW"
+			(at 185.42 124.46 0)
+			(effects
+				(font
+					(size 1.27 1.27)
+				)
+				(hide yes)
 			)
 		)

Commit message: fix MPN of 110K resistors
Parts:
- R12: MPN 0805W8F1002T5E -> 0805W8F1103T5E
Changed lines of the file:
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@@
 			)
 		)
-		(property "MPN" "0805W8F1002T5E"
+		(property "MPN" "0805W8F1103T5E"
 			(at 210.82 135.89 0)
 			(effects

Commit message: Add  Title block to other sheets
Other:
- company: (none) -> MicroRidge Technology LTD
- title: (none) -> FMC-SFP
Changed lines of the file:
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@@
 	(generator_version "8.0")
 	(paper "A4")
+	(title_block
+		(title "FMC-SFP")
+		(date "2024-08-06")
+		(rev "Rev1-2-g26e7d07")
+		(company "MicroRidge Technology LTD")
+	)
 	(junction
 		(at 62.23 48.26)
